Commit message: chore: snapshot visuals and motion diagnostics before native-only rollback

File: Dummy上位机/resources/models/DummyRobot_URDF/urdf/DummyRobot_URDF.urdf (robot description, URDF)
Before this commit: robot DummyRobot_URDF, 10 links, 9 joints
Links:
- link base_link: geometry collision mesh filename=package://DummyRobot_URDF/meshes/base_link.STL; visual mesh filename=package://DummyRobot_URDF/meshes/base_link.STL

Commit message: chore(host): snapshot before unified operation status

File: Dummy上位机/resources/models/DummyRobot_URDF/urdf/DummyRobot_URDF.urdf (robot description, URDF)
Before this commit: robot DummyRobot_URDF, 10 links, 9 joints
Links:
- added link base_rail_control; collision mesh filename=package://DummyRobot_URDF/meshes/base_rail_control.stl; visual mesh filename=package://DummyRobot_URDF/meshes/base_rail_control.stl
Joints:
- added joint base_rail_control_fixed: type fixed, parent base_rail, child base_rail_control, origin xyz=0 0 0 rpy=0 0 0
